Commit message: working version with ur_mount

File: ur_moveit_config/srdf/ur.srdf.xacro (robot description, xacro)
@@ -7,3 +7,7 @@
   <xacro:include filename="$(find ur_moveit_config)/srdf/ur_macro.srdf.xacro"/>
   <xacro:ur_srdf name="$(arg name)" prefix="$(arg prefix)"/>
+  <virtual_joint name="world_joint"
+                type="fixed"
+                parent_frame="world"
+                child_link="ur_mount"/>
 </robot>

File: ur_robot_driver/urdf/ur_with_custom.urdf.xacro (robot description, xacro)
@@ -43,9 +43,10 @@
   <!-- Include macro using the passed absolute path -->
   <xacro:include filename="$(arg ur_description_share)/urdf/ur_macro.xacro"/>
-  <link name="world"/>
+  <!-- <link name="world"/> -->
+  <link name="ur_mount"/>
   <xacro:ur_robot
       name="$(arg name)"
       tf_prefix="$(arg tf_prefix)"
-      parent="world"
+      parent="ur_mount"
       joint_limits_parameters_file="$(arg joint_limit_params)"
       kinematics_parameters_file="$(arg kinematics_params)"
